Commit message: Set Gazebo max_force via dynamics friction attr

File: urdf/ur_macro.xacro (robot description, xacro)
@@ -272,5 +272,11 @@
          <safety_controller soft_lower_limit="${shoulder_pan_lower_limit + safety_pos_margin}" soft_upper_limit="${shoulder_pan_upper_limit - safety_pos_margin}" k_position="${safety_k_position}" k_velocity="0.0"/>
       </xacro:if>
-      <dynamics damping="0" friction="0"/>
+      <!-- For ODE physics engine, see https://github.com/UniversalRobots/Universal_Robots_ROS2_Gazebo_Simulation/issues/19#issuecomment-1481372879 -->
+      <xacro:if value="${sim_gazebo}">
+        <dynamics damping="0" friction="${shoulder_pan_effort_limit*100.0}"/>
+      </xacro:if>
+      <xacro:unless value="${sim_gazebo}">
+        <dynamics damping="0" friction="0"/>
+      </xacro:unless>
     </joint>
     <joint name="${prefix}shoulder_lift_joint" type="revolute">
@@ -284,5 +290,11 @@
          <safety_controller soft_lower_limit="${shoulder_lift_lower_limit + safety_pos_margin}" soft_upper_limit="${shoulder_lift_upper_limit - safety_pos_margin}" k_position="${safety_k_position}" k_velocity="0.0"/>
       </xacro:if>
-      <dynamics damping="0" friction="0"/>
+      <!-- For ODE physics engine, see https://github.com/UniversalRobots/Universal_Robots_ROS2_Gazebo_Simulation/issues/19#issuecomment-1481372879 -->
+      <xacro:if value="${sim_gazebo}">
+        <dynamics damping="0" friction="${shoulder_lift_effort_limit*100.0}"/>
+      </xacro:if>
+      <xacro:unless value="${sim_gazebo}">
+        <dynamics damping="0" friction="0"/>
+      </xacro:unless>
     </joint>
     <joint name="${prefix}elbow_joint" type="revolute">
@@ -296,5 +308,11 @@
          <safety_controller soft_lower_limit="${elbow_joint_lower_limit + safety_pos_margin}" soft_upper_limit="${elbow_joint_upper_limit - safety_pos_margin}" k_position="${safety_k_position}" k_velocity="0.0"/>
       </xacro:if>
-      <dynamics damping="0" friction="0"/>
+      <!-- For ODE physics engine, see https://github.com/UniversalRobots/Universal_Robots_ROS2_Gazebo_Simulation/issues/19#issuecomment-1481372879 -->
+      <xacro:if value="${sim_gazebo}">
+        <dynamics damping="0" friction="${elbow_joint_effort_limit*100.0}"/>
+      </xacro:if>
+      <xacro:unless value="${sim_gazebo}">
+        <dynamics damping="0" friction="0"/>
+      </xacro:unless>
     </joint>
     <joint name="${prefix}wrist_1_joint" type="revolute">
@@ -308,5 +326,11 @@
          <safety_controller soft_lower_limit="${wrist_1_lower_limit + safety_pos_margin}" soft_upper_limit="${wrist_1_upper_limit - safety_pos_margin}" k_position="${safety_k_position}" k_velocity="0.0"/>
       </xacro:if>
-      <dynamics damping="0" friction="0"/>
+      <!-- For ODE physics engine, see https://github.com/UniversalRobots/Universal_Robots_ROS2_Gazebo_Simulation/issues/19#issuecomment-1481372879 -->
+      <xacro:if value="${sim_gazebo}">
+        <dynamics damping="0" friction="${wrist_1_effort_limit*100.0}"/>
+      </xacro:if>
+      <xacro:unless value="${sim_gazebo}">
+        <dynamics damping="0" friction="0"/>
+      </xacro:unless>
     </joint>
     <joint name="${prefix}wrist_2_joint" type="revolute">
@@ -320,5 +344,11 @@
          <safety_controller soft_lower_limit="${wrist_2_lower_limit + safety_pos_margin}" soft_upper_limit="${wrist_2_upper_limit - safety_pos_margin}" k_position="${safety_k_position}" k_velocity="0.0"/>
       </xacro:if>
-      <dynamics damping="0" friction="0"/>
+      <!-- For ODE physics engine, see https://github.com/UniversalRobots/Universal_Robots_ROS2_Gazebo_Simulation/issues/19#issuecomment-1481372879 -->
+      <xacro:if value="${sim_gazebo}">
+        <dynamics damping="0" friction="${wrist_2_effort_limit*100.0}"/>
+      </xacro:if>
+      <xacro:unless value="${sim_gazebo}">
+        <dynamics damping="0" friction="0"/>
+      </xacro:unless>
     </joint>
     <joint name="${prefix}wrist_3_joint" type="revolute">
@@ -332,5 +362,11 @@
          <safety_controller soft_lower_limit="${wrist_3_lower_limit + safety_pos_margin}" soft_upper_limit="${wrist_3_upper_limit - safety_pos_margin}" k_position="${safety_k_position}" k_velocity="0.0"/>
       </xacro:if>
-      <dynamics damping="0" friction="0"/>
+      <!-- For ODE physics engine, see https://github.com/UniversalRobots/Universal_Robots_ROS2_Gazebo_Simulation/issues/19#issuecomment-1481372879 -->
+      <xacro:if value="${sim_gazebo}">
+        <dynamics damping="0" friction="${wrist_3_effort_limit*100.0}"/>
+      </xacro:if>
+      <xacro:unless value="${sim_gazebo}">
+        <dynamics damping="0" friction="0"/>
+      </xacro:unless>
     </joint>
     <link name="${prefix}ft_frame"/>

Commit message: Remove shoulder_pan dynamics tag

File: urdf/ur_macro.xacro (robot description, xacro)
@@ -272,5 +272,4 @@
          <safety_controller soft_lower_limit="${shoulder_pan_lower_limit + safety_pos_margin}" soft_upper_limit="${shoulder_pan_upper_limit - safety_pos_margin}" k_position="${safety_k_position}" k_velocity="0.0"/>
       </xacro:if>
-      <dynamics damping="0" friction="0"/>
     </joint>
     <joint name="${prefix}shoulder_lift_joint" type="revolute">
