Commit message: Try overriding joint

File: urdf/ur.urdf.xacro (robot description, xacro)
@@ -89,4 +89,12 @@
     <gazebo reference="world">
     </gazebo>
+    <gazebo reference="$(arg prefix)shoulder_pan_joint">
+      <axis>
+        <dynamics>
+          <damping>0.0</damping>
+          <friction>867530.9</friction>
+        </dynamics>
+      </axis>
+    </gazebo>
     <gazebo>
       <plugin filename="libgazebo_ros2_control.so" name="gazebo_ros2_control">

Commit message: Try springstiffness

File: urdf/ur.urdf.xacro (robot description, xacro)
@@ -90,10 +90,9 @@
     </gazebo>
     <gazebo reference="$(arg prefix)shoulder_pan_joint">
-      <axis>
-        <dynamics>
-          <damping>0.0</damping>
-          <friction>867530.9</friction>
-        </dynamics>
-      </axis>
+      <springStiffness>98756.4</springStiffness>
+      <dynamics>
+        <damping>0.0</damping>
+        <friction>867530.9</friction>
+      </dynamics>
     </gazebo>
     <gazebo>
