Commit message: Possibly working hardware dep injection

File: urdf/inc/ur_common.xacro (robot description, xacro)
@@ -37,5 +37,5 @@
     <mesh filename="${mesh}"/>
   </xacro:macro>
-  <xacro:macro name="read_model_data" params="joint_limits_parameters_file kinematics_parameters_file physical_parameters_file visual_parameters_file force_abs_paths">
+  <xacro:macro name="read_model_data" params="joint_limits_parameters_file kinematics_parameters_file physical_parameters_file visual_parameters_file joint_dynamics_parameters_file force_abs_paths">
     <xacro:property name="force_abs_paths" value="${force_abs_paths}" scope="parent"/>
     <!-- Read .yaml files from disk, load content into properties -->
@@ -44,4 +44,5 @@
     <xacro:property name="config_physical_parameters" value="${xacro.load_yaml(physical_parameters_file)}"/>
     <xacro:property name="config_visual_parameters" value="${xacro.load_yaml(visual_parameters_file)}"/>
+    <xacro:property name="config_joint_dynamics" value="${xacro.load_yaml(joint_dynamics_parameters_file)}"/>
     <!-- Extract subsections from yaml dictionaries -->
     <xacro:property name="sec_limits" value="${config_joint_limit_parameters['joint_limits']}"/>
@@ -51,4 +52,5 @@
     <xacro:property name="sec_mesh_files" value="${config_visual_parameters['mesh_files']}" scope="parent"/>
     <xacro:property name="sec_kinematics" value="${config_kinematics_parameters['kinematics']}" />
+    <xacro:property name="sec_joint_dynamics" value="${config_joint_dynamics['joint_dynamics']}" />
     <!-- JOINTS LIMIT PARAMETERS -->
     <xacro:property name="shoulder_pan_lower_limit" value="${sec_limits['shoulder_pan_joint']['min_position']}" scope="parent"/>
@@ -76,4 +78,17 @@
     <xacro:property name="wrist_3_velocity_limit" value="${sec_limits['wrist_3_joint']['max_velocity']}" scope="parent"/>
     <xacro:property name="wrist_3_effort_limit" value="${sec_limits['wrist_3_joint']['max_effort']}" scope="parent"/>
+    <!-- JOINT DYNAMICS PARAMETERS -->
+    <xacro:property name="shoulder_pan_damping" value="${sec_joint_dynamics['shoulder_pan_joint']['damping']}" scope="parent"/>
+    <xacro:property name="shoulder_pan_friction" value="${sec_joint_dynamics['shoulder_pan_joint']['friction']}" scope="parent"/>
+    <xacro:property name="shoulder_lift_damping" value="${sec_joint_dynamics['shoulder_lift_joint']['damping']}" scope="parent"/>
+    <xacro:property name="shoulder_lift_friction" value="${sec_joint_dynamics['shoulder_lift_joint']['friction']}" scope="parent"/>
+    <xacro:property name="elbow_joint_damping" value="${sec_joint_dynamics['elbow_joint']['damping']}" scope="parent"/>
+    <xacro:property name="elbow_joint_friction" value="${sec_joint_dynamics['elbow_joint']['friction']}" scope="parent"/>
+    <xacro:property name="wrist_1_damping" value="${sec_joint_dynamics['wrist_1_joint']['damping']}" scope="parent"/>
+    <xacro:property name="wrist_1_friction" value="${sec_joint_dynamics['wrist_1_joint']['friction']}" scope="parent"/>
+    <xacro:property name="wrist_2_damping" value="${sec_joint_dynamics['wrist_2_joint']['damping']}" scope="parent"/>
+    <xacro:property name="wrist_2_friction" value="${sec_joint_dynamics['wrist_2_joint']['friction']}" scope="parent"/>
+    <xacro:property name="wrist_3_damping" value="${sec_joint_dynamics['wrist_3_joint']['damping']}" scope="parent"/>
+    <xacro:property name="wrist_3_friction" value="${sec_joint_dynamics['wrist_3_joint']['friction']}" scope="parent"/>
     <!-- DH PARAMETERS -->
     <xacro:property name="d1" value="${sec_dh_parameters['d1']}" scope="parent"/>

File: urdf/ur.ros2_control.xacro (robot description, xacro)
@@ -13,7 +13,7 @@
     <!--<xacro:ur_arm_transmission prefix="${prefix}" hw_interface="${transmission_hw_interface}" />-->
     <ros2_control name="${name}" type="system">
-      <!-- Hardware dependency injection from outside the macro-->
+      <!-- Start hardware dependency injection from outside the macro-->
       <xacro:insert_block name="hardware_system" />
-      <!-- -->
+      <!-- End hardware dependency injection -->
       <joint name="${prefix}shoulder_pan_joint">
         <command_interface name="position">

File: urdf/ur.urdf.xacro (robot description, xacro)
@@ -7,4 +7,6 @@
    <!-- include ros2 control -->
    <xacro:include filename="$(find ur_description)/urdf/ur.ros2_control.xacro" />
+   <!-- include ros2_control hardware instantiation (for now, then migrate later to responsible packages) -->
+   <xacro:include filename="$(find ur_description)/urdf/ur_hardware.xacro"/>
    <!-- possible 'ur_type' values: ur3, ur3e, ur5, ur5e, ur10, ur10e, ur16e -->
    <!-- the default value should raise an error in case this was called without defining the type -->
@@ -16,4 +18,5 @@
    <xacro:arg name="physical_params" default="$(find ur_description)/config/$(arg ur_type)/physical_parameters.yaml"/>
    <xacro:arg name="visual_params" default="$(find ur_description)/config/$(arg ur_type)/visual_parameters.yaml"/>
+   <xacro:arg name="joint_dynamics_params" default="$(find ur_description)/config/$(arg ur_type)/joint_dynamics_parameters.yaml"/>
    <xacro:arg name="transmission_hw_interface" default=""/>
    <xacro:arg name="safety_limits" default="false"/>
@@ -50,7 +53,10 @@
    <xacro:property name="sim_gazebo" default="$(arg sim_gazebo)"/>
    <xacro:property name="sim_ignition" default="$(arg sim_ignition)"/>
+   <xacro:property name="fake_hardware" default="$(arg use_fake_hardware)"/>
    <!-- create link fixed to the "world" -->
    <link name="world" />
    <!-- load model data -->
+   <!-- This puts a bunch of named parameters in the top-level scope which are consumed inside later macros-->
+   <!-- See https://github.com/ros/xacro/pull/105 -->
    <xacro:read_model_data
      joint_limits_parameters_file="$(arg joint_limit_params)"
@@ -58,4 +64,5 @@
      physical_parameters_file="$(arg physical_params)"
      visual_parameters_file="$(arg visual_params)"
+     joint_dynamics_parameters_file="$(arg joint_dynamics_params)"
      force_abs_paths="${sim_gazebo or sim_ignition}"/>
    <!-- arm instance -->
@@ -70,18 +77,55 @@
      <origin xyz="0 0 0" rpy="0 0 0" />          <!-- position robot in the world -->
    </xacro:ur_robot>
-   <!-- ros2 control instance, follow this in your own package, ur_description prepares fake hardware -->
-   <!-- ur_robot_driver would construct the complicated block with all the real hardware parameters -->
+   <!-- ros2 control, if needed -->
+   <!-- ur_description might eventually prepare fake/mock hardware only, delegating the <hardware> block to a consumer package -->
+   <xacro:property name="needs_non_joint_interfaces" value="${not (sim_gazebo or sim_ignition)}"/>
    <xacro:ur_ros2_control
-     name="$(arg name)" prefix="$(arg prefix)"
-     add_non_joint_interfaces="true"
-     initial_positions="${xacro.load_yaml(initial_positions_file)}"
-   >
-      <hardware_system>
-         <hardware>
-            <plugin>mock_components/GenericSystem</plugin>
-            <param name="fake_sensor_commands">$(arg fake_sensor_commands)</param>
-            <param name="state_following_offset">0.0</param>
-         </hardware>
-      </hardware_system>
+      name="$(arg name)" prefix="$(arg prefix)"
+      add_non_joint_interfaces="${needs_non_joint_interfaces}"
+      initial_positions="${xacro.load_yaml(initial_positions_file)}"
+      >
+      <!-- dz: For now, I conditionally pass the right <hardware> as a block param. -->
+      <!-- dz: Later, this wouldn't be necessary, a consumer package could create and pass it in its top-level xacro -->
+         <hardware_system>
+            <xacro:unless value="${sim_gazebo or sim_ignition or fake_hardware}">
+               <xacro:ur_real_hardware_block
+                  headless_mode="$(arg headless_mode)"
+                  initial_positions="${xacro.load_yaml(initial_positions_file)}"
+                  use_tool_communication="$(arg use_tool_communication)"
+                  tool_voltage="$(arg tool_voltage)"
+                  tool_parity="$(arg tool_parity)"
+                  tool_baud_rate="$(arg tool_baud_rate)"
+                  tool_stop_bits="$(arg tool_stop_bits)"
+                  tool_rx_idle_chars="$(arg tool_rx_idle_chars)"
+                  tool_tx_idle_chars="$(arg tool_tx_idle_chars)"
+                  tool_device_name="$(arg tool_device_name)"
+                  tool_tcp_port="$(arg tool_tcp_port)"
+                  robot_ip="$(arg robot_ip)"
+                  script_filename="$(arg script_filename)"
+                  output_recipe_filename="$(arg output_recipe_filename)"
+                  input_recipe_filename="$(arg input_recipe_filename)"
+                  reverse_ip="$(arg reverse_ip)"
+                  script_command_port="$(arg script_command_port)"
+                  transmission_hw_interface="$(arg transmission_hw_interface)"
+               />
+            </xacro:unless>
+            <xacro:if value="${fake_hardware and not (sim_gazebo or sim_ignition)}">
+               <hardware>
+                  <plugin>mock_components/GenericSystem</plugin>
+                  <param name="fake_sensor_commands">$(arg fake_sensor_commands)</param>
+                  <param name="state_following_offset">0.0</param>
+               </hardware>
+            </xacro:if>
+            <xacro:if value="${sim_gazebo}">
+               <hardware>
+                  <plugin>gazebo_ros2_control/GazeboSystem</plugin>
+               </hardware>
+            </xacro:if>
+            <xacro:if value="${sim_ignition}">
+               <hardware>
+                  <plugin>ign_ros2_control/IgnitionSystem</plugin>
+               </hardware>
+            </xacro:if>
+         </hardware_system>
    </xacro:ur_ros2_control>
    <!-- dz: These move to their respective simulation packages -->

File: urdf/ur_macro.xacro (robot description, xacro)
@@ -52,27 +52,5 @@
     safety_pos_margin:=0.15
     safety_k_position:=20
-    use_fake_hardware:=false
-    fake_sensor_commands:=false
-    sim_gazebo:=false
-    sim_ignition:=false
-    headless_mode:=false
-    initial_positions:=${dict(shoulder_pan_joint=0.0,shoulder_lift_joint=-1.57,elbow_joint=0.0,wrist_1_joint=-1.57,wrist_2_joint=0.0,wrist_3_joint=0.0)}
-    use_tool_communication:=false
-    tool_voltage:=0
-    tool_parity:=0
-    tool_baud_rate:=115200
-    tool_stop_bits:=1
-    tool_rx_idle_chars:=1.5
-    tool_tx_idle_chars:=3.5
-    tool_device_name:=/tmp/ttyUR
-    tool_tcp_port:=54321
-    robot_ip:=0.0.0.0
-    script_filename:=to_be_filled_by_ur_robot_driver
-    output_recipe_filename:=to_be_filled_by_ur_robot_driver
-    input_recipe_filename:=to_be_filled_by_ur_robot_driver
-    reverse_port:=50001
-    script_sender_port:=50002
-    reverse_ip:=0.0.0.0
-    script_command_port:=50004">
+    ">
     <!-- links -  main serial chain -->
     <link name="${prefix}base_link"/>
@@ -226,5 +204,5 @@
          <safety_controller soft_lower_limit="${shoulder_pan_lower_limit + safety_pos_margin}" soft_upper_limit="${shoulder_pan_upper_limit - safety_pos_margin}" k_position="${safety_k_position}" k_velocity="0.0"/>
       </xacro:if>
-      <dynamics damping="0" friction="0"/>
+      <dynamics damping="${shoulder_pan_damping}" friction="${shoulder_pan_friction}"/>
     </joint>
     <joint name="${prefix}shoulder_lift_joint" type="revolute">
@@ -238,5 +216,5 @@
          <safety_controller soft_lower_limit="${shoulder_lift_lower_limit + safety_pos_margin}" soft_upper_limit="${shoulder_lift_upper_limit - safety_pos_margin}" k_position="${safety_k_position}" k_velocity="0.0"/>
       </xacro:if>
-      <dynamics damping="0" friction="0"/>
+      <dynamics damping="${shoulder_lift_damping}" friction="${shoulder_lift_friction}"/>
     </joint>
     <joint name="${prefix}elbow_joint" type="revolute">
@@ -250,5 +228,5 @@
          <safety_controller soft_lower_limit="${elbow_joint_lower_limit + safety_pos_margin}" soft_upper_limit="${elbow_joint_upper_limit - safety_pos_margin}" k_position="${safety_k_position}" k_velocity="0.0"/>
       </xacro:if>
-      <dynamics damping="0" friction="0"/>
+      <dynamics damping="${elbow_joint_damping}" friction="${elbow_joint_friction}"/>
     </joint>
     <joint name="${prefix}wrist_1_joint" type="revolute">
@@ -262,5 +240,5 @@
          <safety_controller soft_lower_limit="${wrist_1_lower_limit + safety_pos_margin}" soft_upper_limit="${wrist_1_upper_limit - safety_pos_margin}" k_position="${safety_k_position}" k_velocity="0.0"/>
       </xacro:if>
-      <dynamics damping="0" friction="0"/>
+      <dynamics damping="${wrist_1_damping}" friction="${wrist_1_friction}"/>
     </joint>
     <joint name="${prefix}wrist_2_joint" type="revolute">
@@ -274,5 +252,5 @@
          <safety_controller soft_lower_limit="${wrist_2_lower_limit + safety_pos_margin}" soft_upper_limit="${wrist_2_upper_limit - safety_pos_margin}" k_position="${safety_k_position}" k_velocity="0.0"/>
       </xacro:if>
-      <dynamics damping="0" friction="0"/>
+      <dynamics damping="${wrist_2_damping}" friction="${wrist_2_friction}"/>
     </joint>
     <joint name="${prefix}wrist_3_joint" type="revolute">
@@ -286,5 +264,5 @@
          <safety_controller soft_lower_limit="${wrist_3_lower_limit + safety_pos_margin}" soft_upper_limit="${wrist_3_upper_limit - safety_pos_margin}" k_position="${safety_k_position}" k_velocity="0.0"/>
       </xacro:if>
-      <dynamics damping="0" friction="0"/>
+      <dynamics damping="${wrist_3_damping}" friction="${wrist_3_friction}"/>
     </joint>
     <link name="${prefix}ft_frame"/>
